File: hardware/trappy/trappy.kicad_pcb (KiCad board)
At the start: 2 copper layers, 65 x 56 mm, 43 parts, among them J1 Screw_Terminal_01x02, J10 STRIP0, J11 STRIP9, J12 STRIP10, J13 STRIP11, J14 STRIP12, J15 STRIP13, J16 STRIP14, J17 STRIP15, J18 RPI POWER JMP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

Commit message: Looking pretty good!
Parts:
- added G***: LOGO, mayhem:mayhem_logo_tiny, F.Cu at (123.5, 86.0)
- J18: value RPI POWER JMP -> Power RPi
- moved J18 2.63 mm to (121.4, 74.5)
Routing:
- net /STRIP11: track 0.00 -> 38.5 mm, vias 0 -> 2
- net /SHIFT13: track 0.00 -> 31.7 mm, vias 0 -> 2
- net /SHIFT14: track 19.8 -> 47.8 mm, vias 1 -> 3
- net /SHIFT4: track 0.00 -> 27.4 mm, vias 0 -> 3
- net /SHIFT5: track 0.00 -> 26.9 mm, vias 0 -> 1
- net /STRIP10: track 0.00 -> 25.3 mm, vias 0 -> 2
- net /SHIFT0: track 0.00 -> 23.8 mm, vias 0 -> 1
- net /STRIP7: track 0.00 -> 23.3 mm, vias 0 -> 2
- net /STRIP0: track 0.00 -> 22.9 mm, vias 0 -> 2
- net /STRIP12: track 0.00 -> 21.4 mm
- net /SHIFT9: track 0.00 -> 21.1 mm, vias 0 -> 2
- net /SHIFT1: track 0.00 -> 18.1 mm, vias 0 -> 2
- net /SHIFT15: track 28.4 -> 46.2 mm, vias 0 -> 2
- net /SHIFT2: track 0.00 -> 17.2 mm, vias 0 -> 2
- net /SHIFT10: track 0.00 -> 17.2 mm
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Other:
- outline, holes or cut-outs redrawn
- board text added: "5V"
- board text added: "Add jumper to"
- board text added: "GND"
- board text added: "from 5V"
