File: hardware/trappy/trappy.kicad_sch (KiCad schematic)
At the start: 39 parts, among them J1 Screw_Terminal_01x02, J10 STRIP0, J11 STRIP9, J12 STRIP10, J13 STRIP11, J14 STRIP12, J15 STRIP13, J16 STRIP14, J17 STRIP15, J18 RPI POWER JMP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

Commit message: Looking pretty good!
Changed lines of the file:
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@@
 		(dnp no)
 		(fields_autoplaced yes)
-		(property "Reference" "J2"
-			(at 141.8941 102.87 0)
-			(effects
-				(font
-					(size 1.27 1.27)
-				)
-				(justify left)
-			)
-		)
 		(property "Value" "RPi"
 			(at 141.8941 105.41 0)
