File: hardware/trappy.kicad_pcb (KiCad board)
At the start: 2 copper layers, 65 x 56 mm, 44 parts, among them J1 Screw_Terminal_01x02, J10 STRIP0, J11 STRIP9, J12 STRIP10, J13 STRIP11, J14 STRIP12, J15 STRIP13, J16 STRIP14, J17 STRIP15, J18 Power RPi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

Commit message: Check in latest trappy board, awaiting the board from china
Parts:
- J18: value Power RPi -> RPI POWER JMP
- U1, U2, U3, U4: value SN74AHCT125RGYR -> SN74AHCT125PWR; footprint Package_DFN_QFN:Texas_S-PVQFN-N14 -> Package_SO:TSSOP-14_4.4x5mm_P0.65mm
- moved U3 3.94 mm to (135.5, 79.4), turned to 0 degrees
- moved U1 2.94 mm to (147.5, 79.4)
- moved U2 1.20 mm to (159.5, 79.4)
- moved U4 1.18 mm to (171.5, 79.4)
- moved G*** 0.15 mm to (123.7, 85.9)
Routing:
- net /STRIP11: track 38.5 -> 19.1 mm, vias 2 -> 0
- net /STRIP10: track 25.3 -> 12.8 mm, vias 2 -> 0
- net /SHIFT13: track 31.7 -> 21.8 mm
- net /SHIFT11: track 63.0 -> 72.5 mm, vias 0 -> 2
- net /SHIFT14: track 47.8 -> 38.9 mm, vias 3 -> 1
- net /STRIP9: track 13.3 -> 18.7 mm
- net /SHIFT4: track 27.4 -> 22.8 mm, vias 3 -> 1
- net /SHIFT12: track 14.2 -> 18.6 mm
- net /SHIFT5: track 26.9 -> 22.7 mm
- net /STRIP8: track 10.9 -> 14.9 mm
- net /SHIFT9: track 21.1 -> 17.8 mm, vias 2 -> 1
- net /GND: track 31.5 -> 28.8 mm
- net /STRIP5: track 11.8 -> 14.2 mm
- net /SHIFT10: track 17.2 -> 19.4 mm, vias 0 -> 2
- net /SHIFT8: track 58.6 -> 56.3 mm, vias 2 -> 0
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Other:
- board text added: "(c) Mayhem & Chaos 2024"
- board text added: "LED"
- board text added: "Power RPi"
- board text added: "RPi WS2812/3 SMI LED Driver Board v2024-05-17"
- board text added: "STRIP0"
- board text added: "STRIP1"
- board text added: "STRIP10"
- board text added: "STRIP11"
- board text added: "STRIP12"
- board text added: "STRIP13"
- board text added: "STRIP14"
- board text added: "STRIP15"
- board text added: "STRIP2"
- board text added: "STRIP3"
- board text added: "STRIP4"
- board text added: "STRIP6"
- board text added: "STRIP7"
- board text added: "STRIP8"
- board text added: "STRIP9"
