File: hardware/trappy.kicad_sch (KiCad schematic)
At the start: 39 parts, among them J1 Screw_Terminal_01x02, J10 STRIP0, J11 STRIP9, J12 STRIP10, J13 STRIP11, J14 STRIP12, J15 STRIP13, J16 STRIP14, J17 STRIP15, J18 RPI POWER JMP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

Commit message: Check in latest trappy board, awaiting the board from china
Parts:
- U1, U2, U3, U4: value SN74AHCT125RGYR -> SN74AHCT125PWR; footprint Package_DFN_QFN:Texas_S-PVQFN-N14 -> Package_SO:TSSOP-14_4.4x5mm_P0.65mm
Changed lines of the file:
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@@
 			)
 		)
-		(property "Value" "SN74AHCT125RGYR"
+		(property "Value" "SN74AHCT125PWR"
 			(at 211.7441 125.73 0)
 			(effects
@@
 			)
 		)
-		(property "Footprint" "Package_DFN_QFN:Texas_S-PVQFN-N14"
+		(property "Footprint" "Package_SO:TSSOP-14_4.4x5mm_P0.65mm"
 			(at 209.55 142.24 0)
 			(effects
@@
 		(dnp no)
 		(fields_autoplaced yes)
+		(property "Reference" "J2"
+			(at 139.7 69.85 0)
+			(effects
+				(font
+					(size 1.27 1.27)
+				)
+				(hide yes)
+			)
+		)
 		(property "Value" "RPi"
 			(at 141.8941 105.41 0)
@@
 			)
 		)
-		(property "Value" "SN74AHCT125RGYR"
+		(property "Value" "SN74AHCT125PWR"
 			(at 51.7241 125.73 0)
 			(effects
@@
 			)
 		)
-		(property "Footprint" "Package_DFN_QFN:Texas_S-PVQFN-N14"
+		(property "Footprint" "Package_SO:TSSOP-14_4.4x5mm_P0.65mm"
 			(at 49.53 142.24 0)
 			(effects
@@
 		(on_board yes)
 		(dnp no)
-		(fields_autoplaced yes)
 		(property "Reference" "U2"
 			(at 103.7941 123.19 0)
@@
 			)
 		)
-		(property "Value" "SN74AHCT125RGYR"
+		(property "Value" "SN74AHCT125PWR"
 			(at 103.7941 125.73 0)
 			(effects
@@
 			)
 		)
-		(property "Footprint" "Package_DFN_QFN:Texas_S-PVQFN-N14"
+		(property "Footprint" "Package_SO:TSSOP-14_4.4x5mm_P0.65mm"
 			(at 101.6 142.24 0)
 			(effects
@@
 			)
 		)
-		(property "Value" "SN74AHCT125RGYR"
+		(property "Value" "SN74AHCT125PWR"
 			(at 157.1341 125.73 0)
 			(effects
@@
 			)
 		)
-		(property "Footprint" "Package_DFN_QFN:Texas_S-PVQFN-N14"
+		(property "Footprint" "Package_SO:TSSOP-14_4.4x5mm_P0.65mm"
 			(at 154.94 142.24 0)
 			(effects
